File: hardware/epaperle.sch (KiCad schematic (older format))
At the start: 29 parts, among them IC1 BLE112-A, P1 CONN_5, Q1 Si1304BDL, Q2 Q_PMOS_GSD, U2 GDE021A1

Commit message: bom fixes
Parts:
- D1, D2, D3: value MBR0530 -> MBR180S1-7
- Q1: value Si1304BDL -> PMF250XNE
- Q2: value Q_PMOS_GSD -> DMG1013UWQ
Changed lines of the file:
@@
 P 7600 1675
 F 0 "D1" H 7600 1775 40  0000 C CNN
-F 1 "MBR0530" H 7600 1575 40  0000 C CNN
+F 1 "MBR180S1-7" H 7600 1575 40  0000 C CNN
 F 2 "Diodes_SMD:D_SOD-123" H 7600 1675 60  0001 C CNN
 F 3 "" H 7600 1675 60  0000 C CNN
@@
 P 7650 925
 F 0 "D2" H 7650 1025 40  0000 C CNN
-F 1 "MBR0530" H 7650 825 40  0000 C CNN
+F 1 "MBR180S1-7" V 7550 700 40  0000 C CNN
 F 2 "Diodes_SMD:D_SOD-123" H 7650 925 60  0001 C CNN
 F 3 "" H 7650 925 60  0000 C CNN
@@
 P 7650 1325
 F 0 "D3" H 7650 1425 40  0000 C CNN
-F 1 "MBR0530" H 7650 1225 40  0000 C CNN
+F 1 "MBR180S1-7" V 7550 1100 40  0000 C CNN
 F 2 "Diodes_SMD:D_SOD-123" H 7650 1325 60  0001 C CNN
 F 3 "" H 7650 1325 60  0000 C CNN
@@
 P 7000 1925
 F 0 "Q1" H 7010 2095 60  0000 R CNN
-F 1 "Si1304BDL" H 7125 1650 60  0000 R CNN
+F 1 "PMF250XNE" H 7000 1725 60  0000 R CNN
 F 2 "TO_SOT_Packages_SMD:SOT-323_SC-70" H 7000 1925 60  0001 C CNN
 F 3 "" H 7000 1925 60  0000 C CNN
@@
 P 4275 1675
 F 0 "Q2" H 4481 1721 50  0000 L CNN
-F 1 "Q_PMOS_GSD" H 4481 1630 50  0000 L CNN
+F 1 "DMG1013UWQ" H 4481 1630 50  0000 L CNN
 F 2 "TO_SOT_Packages_SMD:SOT-323_SC-70" H 4475 1775 50  0001 C CNN
 F 3 "" H 4275 1675 50  0001 C CNN
